Commit message: enme480 changes

File: urdf/ur.urdf.xacro (robot description, xacro)
@@ -4,8 +4,8 @@
    <xacro:arg name="name" default="ur"/>
    <!-- import main macro -->
-   <xacro:include filename="$(find ur_description)/urdf/ur_macro.xacro"/>
+   <xacro:include filename="$(find ur_description)/urdf/enme480_ik.xacro"/>
    <!-- possible 'ur_type' values: ur3, ur3e, ur5, ur5e, ur10, ur10e, ur16e, ur20, ur30 -->
    <!-- the default value should raise an error in case this was called without defining the type -->
-   <xacro:arg name="ur_type" default="ur5x"/>
+   <xacro:arg name="ur_type" default="ur3e"/>
    <!-- parameters -->
    <xacro:arg name="tf_prefix" default="" />
@@ -49,32 +49,6 @@
    <!-- convert to property to use substitution in function -->
    <xacro:property name="initial_positions_file" default="$(arg initial_positions_file)"/>
-   <xacro:property name="is_sim_gazebo" value="$(arg sim_gazebo)"/>
-   <xacro:property name="is_sim_ignition" value="$(arg sim_ignition)"/>
    <!-- create link fixed to the "world" -->
    <link name="world" />
-   <xacro:if value="${is_sim_gazebo or is_sim_ignition}">
-     <link name="ground_plane">
-       <visual>
-         <origin rpy="0 0 0" xyz="0 0 0"/>
-         <geometry>
-           <box size="5 5 0"/>
-         </geometry>
-         <material name="ground_white">
-           <color rgba="1 1 1 0.5"/>
-         </material>
-       </visual>
-       <collision>
-         <origin rpy="0 0 0" xyz="0 0 0"/>
-         <geometry>
-           <box size="5 5 0"/>
-         </geometry>
-       </collision>
-     </link>
-     <joint name="ground_plane_joint" type="fixed">
-       <origin xyz="0 0 -0.01" rpy="0 0 0"/>
-       <parent link="world"/>
-       <child link="ground_plane"/>
-     </joint>
-   </xacro:if>
    <!-- arm -->
    <xacro:ur_robot
@@ -115,5 +89,5 @@
      trajectory_port="$(arg trajectory_port)"
      >
-     <origin xyz="0 0 0" rpy="0 0 0" />          <!-- position robot in the world -->
+     <origin xyz="-0.15 0.15 0" rpy="0 0 0" />          <!-- position robot in the world -->
    </xacro:ur_robot>
    <xacro:if value="$(arg sim_gazebo)">
